File: Kicad/Flashlight_TOF_board/Flashlight_TOF_board.kicad_sch (KiCad schematic)
At the start: 8 parts, among them IC1 PI4ULS3V204ZBEX, IC2 LDK130M18RY, U1 VL53L8CXV0GC_1

Commit message: TOF finished
Parts:
- added C6, C7, C9: 100nF, Capacitor_SMD:C_0805_2012Metric_Pad1.18x1.45mm_HandSolder, symbol Device:C
- added C8: 4uF7, Capacitor_SMD:C_0805_2012Metric_Pad1.18x1.45mm_HandSolder, symbol Device:C
- added IC3: PI4ULS3V204ZBEX, SamacSys_Parts:PI4ULS3V204ZBEX, symbol SamacSys_Parts:PI4ULS3V204ZBEX
- added J1: F52R-1A7H1-11008, SamacSys_Parts:F52R1A7H111008, symbol SamacSys_Parts:F52R-1A7H1-11008
- added R1, R2, R3, R4, R7: 47K, Resistor_SMD:R_0805_2012Metric_Pad1.20x1.40mm_HandSolder, symbol Device:R
- added R5, R6: 2K2, Resistor_SMD:R_0805_2012Metric_Pad1.20x1.40mm_HandSolder, symbol Device:R
- added TP1, TP2, TP3, TP4: WELD, TestPoint:TestPoint_Pad_2.0x2.0mm, symbol Connector:TestPoint
- added TP5: SDA_test, TestPoint:TestPoint_Pad_D2.0mm, symbol Connector:TestPoint
- added TP6: SCL_test, TestPoint:TestPoint_Pad_D2.0mm, symbol Connector:TestPoint
- added TP8: 1V8_test, TestPoint:TestPoint_Pad_D2.0mm, symbol Connector:TestPoint
- C1, C2, C3, C4, C5: value C -> 100nF; footprint (none) -> Capacitor_SMD:C_0805_2012Metric_Pad1.18x1.45mm_HandSolder
- IC1: footprint PI4ULS3V204ZBEX -> SamacSys_Parts:PI4ULS3V204ZBEX
- IC2: footprint SOT95P280X145-5N -> SamacSys_Parts:SOT95P280X145-5N
- U1: footprint VL53L8CXV0GC1 -> SamacSys_Parts:VL53L8CXV0GC1
Connections:
- net +1V8: now also C3.1, U1.A3 (IOVDD), U1.B7 (CORE_1V8), C7.1, C9.2, IC3.14 (VCCB), IC3.8 (EN), R1.2, R2.2, R3.2, R5.2, R6.2, TP8.1; no longer C2.1
- net +3V3: now also U1.C4 (VDD), C6.1, C8.1, IC3.1 (VCCA), J1.7
- net GND: now also IC1.15 (EP), U1.A6 (SWD_IO), U1.A7 (SWD_CLK), U1.C6 (ATEST1), U1.C7 (GND_3), C6.2, C7.2, C8.2, C9.1, IC3.15 (EP), IC3.7 (GND), J1.8, R4.2, R7.2
- net DUT_INT: now reaches U1.A1 (INT_2)
- net DUT_INT: now also IC1.11 (B3), R5.1
- net at U1.A2 (XSHUT): now also R2.1
- net DUT_SDA: now reaches U1.A4 (MOSI)
- net DUT_SDA: now also IC1.12 (B2), R3.1
- net DUT_SCLCK: now reaches U1.A5 (MCLK)
- net DUT_SCLCK: now also IC1.13 (B1), R1.1
- net DUT_SYNC: now reaches U1.B1 (SYNC)
- net DUT_SYNC: now also IC1.10 (B4), R6.1
- net DUT_I2C_RESET: now reaches U1.C1 (SPI_I2C_N)
- net DUT_I2C_RESET: now also IC3.13 (B1), R4.1
- net DUT_NCS: now reaches U1.C2 (NCS)
- net DUT_NCS: now also IC3.12 (B2), R7.1
- net SCLCK: now reaches IC1.2 (A1)
- net SCLCK: now also J1.1, TP6.1
- net SDA: now reaches IC1.3 (A2)
- net SDA: now also J1.2, TP5.1
- net INT: now reaches IC1.4 (A3)
- net INT: now also J1.3
- net SYNC: now reaches IC1.5 (A4)
- net SYNC: now also J1.4
- net at IC2.4 (BYP/ADJ): now also C2.1; no longer C3.1
- new net I2C_RESET: IC3.2 (A1), J1.5
- new net NCS: IC3.3 (A2), J1.6
- no-connect marks 2 -> 18
Other:
- moved on the sheet: IC1, IC2, U1
